File: Eagle/sprite.sch (EAGLE design)
At the start: 40 parts

Commit message: Battery Sprite
Parts:
- removed GNDPIN, VCCPIN: SPRITE_PIN, SpritePin:SPRITE_PIN
- removed TRISOL3, TRISOL4: TRISOLX-WING, TriSolX_QzQube:TRISOLX-WING
- added U$1: CR202, CR202:CR202
Connections:
- net GND: now also U$1.VCC; no longer GNDPIN.P$1, TRISOL3.A, TRISOL4.A
- net VCC: now also U$1.GND, U$1.GND1; no longer TRISOL3.C, TRISOL4.C, VCCPIN.P$1
Other:
- note added: "The board features two TriSolX solar panels, along with a CR2032 coin-cell battery and a set of inductive coils for inductive powering. The inductive coils double as torque coils, controlled via four of the CC430 pins connected to an H-bridge."
- note added: "TriSolX Solar Panels and CR2032"
- note removed: "The board features four TriSolX solar panels, along with a set of inductive coils and a full bridge rectifier for inductive powering. The inductive coils double as torque coils, controlled via four of the CC430 pins connected to an H-bridge."
- note removed: "TriSolX Solar Panels"
Changed lines of the file:
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@@
 <part name="GND22" library="SparkFun" deviceset="GND" device=""/>
 <part name="32KHZ" library="SpriteCrystal" deviceset="SPRITECRYSTAL" device="SPRITECRYSTAL"/>
-<part name="VCCPIN" library="SpritePin" deviceset="SPRITE_PIN" device=""/>
-<part name="GNDPIN" library="SpritePin" deviceset="SPRITE_PIN" device=""/>
-<part name="GND26" library="SparkFun" deviceset="GND" device=""/>
-<part name="P+17" library="SparkFun" deviceset="VCC" device=""/>
 <part name="JP3" library="SparkFun" deviceset="M02" device="PTH"/>
 <part name="R7" library="SparkFun" deviceset="RESISTOR" device="0805-RES" value="56K"/>
@@
 <part name="P+19" library="SparkFun" deviceset="VCC" device=""/>
 <part name="GND30" library="SparkFun" deviceset="GND" device=""/>
-<part name="TRISOL4" library="TriSolX_QzQube" deviceset="TRISOLX-WING" device=""/>
-<part name="P+20" library="SparkFun" deviceset="VCC" device=""/>
-<part name="GND31" library="SparkFun" deviceset="GND" device=""/>
-<part name="TRISOL3" library="TriSolX_QzQube" deviceset="TRISOLX-WING" device=""/>
-<part name="P+21" library="SparkFun" deviceset="VCC" device=""/>
-<part name="GND32" library="SparkFun" deviceset="GND" device=""/>
 <part name="RECTIFIER" library="NSR1030QMUTAG" deviceset="NSR1030QMUTAG" device=""/>
 <part name="H-BRIDGE" library="lv8417cs" deviceset="LV8417CS" device=""/>
@@
 <part name="C12" library="SparkFun" deviceset="CAP" device="0805" value="10uF"/>
 <part name="GND20" library="SparkFun" deviceset="GND" device=""/>
+<part name="U$1" library="CR202" deviceset="CR202" device=""/>
+<part name="P+11" library="SparkFun" deviceset="VCC" device=""/>
+<part name="P+17" library="SparkFun" deviceset="VCC" device=""/>
+<part name="GND13" library="SparkFun" deviceset="GND" device=""/>
 </parts>
 <sheets>
@@
 dipole antennae.</text>
 <text x="256.54" y="53.34" size="5.08" layer="97">Power/Attitude Control:</text>
-<text x="269.24" y="33.02" size="1.778" layer="97">The board features four TriSolX solar panels,
-along with a set of inductive coils and a full bridge
-rectifier for inductive powering. The
+<text x="269.24" y="33.02" size="1.778" layer="97">The board features two TriSolX solar panels,
+along with a CR2032 coin-cell battery and a set
+of inductive coils for inductive powering. The
 inductive coils double as torque coils, controlled
 via four of the CC430 pins connected to an
 H-bridge.</text>
 <text x="38.1" y="38.1" size="2.54" layer="97">Antennae</text>
-<text x="302.26" y="137.16" size="2.54" layer="97">TriSolX Solar Panels</text>
+<text x="292.1" y="137.16" size="2.54" layer="97">TriSolX Solar Panels and CR2032</text>
 <text x="297.18" y="248.92" size="2.54" layer="97">Inductive Powering/Torque Coils</text>
 <text x="292.1" y="7.62" size="2.54" layer="97">Hunter Adams
@@
 <instance part="GND22" gate="1" x="347.98" y="180.34" rot="R180"/>
 <instance part="32KHZ" gate="G$1" x="132.08" y="116.84" rot="R90"/>
-<instance part="VCCPIN" gate="G$1" x="187.96" y="83.82" rot="R270"/>
-<instance part="GNDPIN" gate="G$1" x="198.12" y="83.82" rot="R270"/>
-<instance part="GND26" gate="1" x="198.12" y="106.68" rot="R180"/>
-<instance part="P+17" gate="1" x="187.96" y="104.14"/>
 <instance part="JP3" gate="G$1" x="205.74" y="43.18" rot="R180"/>
 <instance part="R7" gate="G$1" x="198.12" y="53.34" rot="R270"/>
@@
 <instance part="P+19" gate="1" x="292.1" y="127"/>
 <instance part="GND30" gate="1" x="292.1" y="78.74"/>
-<instance part="TRISOL4" gate="G$1" x="337.82" y="99.06" rot="R90"/>
-<instance part="P+20" gate="1" x="337.82" y="127"/>
-<instance part="GND31" gate="1" x="337.82" y="78.74"/>
-<instance part="TRISOL3" gate="G$1" x="322.58" y="99.06" rot="R90"/>
-<instance part="P+21" gate="1" x="322.58" y="127"/>
-<instance part="GND32" gate="1" x="322.58" y="78.74"/>
 <instance part="RECTIFIER" gate="G$1" x="330.2" y="162.56" rot="R180"/>
 <instance part="H-BRIDGE" gate="G$1" x="317.5" y="203.2" rot="R270"/>
@@
 <instance part="C12" gate="G$1" x="302.26" y="223.52" rot="R90"/>
 <instance part="GND20" gate="1" x="287.02" y="223.52" rot="R270"/>
+<instance part="U$1" gate="G$1" x="340.36" y="104.14"/>
+<instance part="P+11" gate="1" x="332.74" y="83.82" rot="R180"/>
+<instance part="P+17" gate="1" x="347.98" y="83.82" rot="R180"/>
+<instance part="GND13" gate="1" x="340.36" y="129.54" rot="R180"/>
 </instances>
 <busses>
@@
 </segment>
 <segment>
-<pinref part="GND26" gate="1" pin="GND"/>
-<pinref part="GNDPIN" gate="G$1" pin="P$1"/>
-<wire x1="198.12" y1="104.14" x2="198.12" y2="83.82" width="0.1524" layer="91"/>
-</segment>
-<segment>
 <pinref part="TRISOL2" gate="G$1" pin="A"/>
 <pinref part="GND29" gate="1" pin="GND"/>
@@
 <pinref part="GND30" gate="1" pin="GND"/>
 <wire x1="292.1" y1="93.98" x2="292.1" y2="81.28" width="0.1524" layer="91"/>
-</segment>
-<segment>
-<pinref part="TRISOL4" gate="G$1" pin="A"/>
-<pinref part="GND31" gate="1" pin="GND"/>
-<wire x1="337.82" y1="93.98" x2="337.82" y2="81.28" width="0.1524" layer="91"/>
-</segment>
-<segment>
-<pinref part="TRISOL3" gate="G$1" pin="A"/>
-<pinref part="GND32" gate="1" pin="GND"/>
-<wire x1="322.58" y1="93.98" x2="322.58" y2="81.28" width="0.1524" layer="91"/>
 </segment>
 <segment>
@@
 <pinref part="C12" gate="G$1" pin="1"/>
 <wire x1="289.56" y1="223.52" x2="297.18" y2="223.52" width="0.1524" layer="91"/>
+</segment>
+<segment>
+<pinref part="GND13" gate="1" pin="GND"/>
+<pinref part="U$1" gate="G$1" pin="VCC"/>
+<wire x1="340.36" y1="127" x2="340.36" y2="124.46" width="0.1524" layer="91"/>
 </segment>
 </net>
@@
 </segment>
 <segment>
-<pinref part="P+20" gate="1" pin="VCC"/>
-<pinref part="TRISOL4" gate="G$1" pin="C"/>
-<wire x1="337.82" y1="127" x2="337.82" y2="104.14" width="0.1524" layer="91"/>
-</segment>
-<segment>
-<pinref part="P+21" gate="1" pin="VCC"/>
-<pinref part="TRISOL3" gate="G$1" pin="C"/>
-<wire x1="322.58" y1="127" x2="322.58" y2="104.14" width="0.1524" layer="91"/>
-</segment>
-<segment>
 <pinref part="P+13" gate="1" pin="VCC"/>
 <pinref part="H-BRIDGE" gate="G$1" pin="VCC"/>
@@
 </segment>
 <segment>
+<pinref part="U$1" gate="G$1" pin="GND1"/>
 <pinref part="P+17" gate="1" pin="VCC"/>
-<pinref part="VCCPIN" gate="G$1" pin="P$1"/>
-<wire x1="187.96" y1="104.14" x2="187.96" y2="83.82" width="0.1524" layer="91"/>
+<wire x1="347.98" y1="86.36" x2="347.98" y2="83.82" width="0.1524" layer="91"/>
+</segment>
+<segment>
+<pinref part="U$1" gate="G$1" pin="GND"/>
+<pinref part="P+11" gate="1" pin="VCC"/>
+<wire x1="332.74" y1="86.36" x2="332.74" y2="83.82" width="0.1524" layer="91"/>
 </segment>
 </net>
